File: breadBoard Power.kicad_pcb (KiCad board)
At the start: 2 copper layers, 53 x 24.5 mm, 13 parts, among them J1 Barrel_Jack, J2 Conn_02x02_Odd_Even, J3 Conn_02x02_Odd_Even, U1 AZ1117-3.3, U2 AZ1117-5.0

Commit message: Add files via upload
Other:
- rule pad_to_mask_clearance: 0.051 -> 0.0762
- rule solder_mask_min_width: 0.25 -> 0.1016
- board text added: "Design by-Razanul Islam Bread Board Power Supply"
Changed lines of the file:
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@@
   (general
     (thickness 1.6)
-    (drawings 17)
+    (drawings 20)
     (tracks 70)
     (zones 0)
@@
     (last_trace_width 0.25)
     (trace_clearance 0.2)
-    (zone_clearance 0.508)
+    (zone_clearance 0.2)
     (zone_45_only no)
     (trace_min 0.2)
@@
     (pad_size 1.524 1.524)
     (pad_drill 0.762)
-    (pad_to_mask_clearance 0.051)
-    (solder_mask_min_width 0.25)
+    (pad_to_mask_clearance 0.0762)
+    (solder_mask_min_width 0.1016)
     (aux_axis_origin 0 0)
-    (visible_elements FFFFFF7F)
+    (visible_elements 7FFFFFFF)
     (pcbplotparams
       (layerselection 0x010fc_ffffffff)
@@
     )
   )
+  (gr_text "Design by-Razanul Islam\nBread Board Power Supply" (at 171.75 90.5) (layer B.SilkS)
+    (effects (font (size 0.5 0.5) (thickness 0.1) italic) (justify mirror))
+  )
+  (dimension 53.00059 (width 0.15) (layer Dwgs.User)
+    (gr_text "2.0866 in" (at 152.225 97.924897 359.7297389) (layer Dwgs.User)
+      (effects (font (size 1 1) (thickness 0.15)))
+    )
+    (feature1 (pts (xy 178.75 92.75) (xy 178.728366 97.336325)))
+    (feature2 (pts (xy 125.75 92.5) (xy 125.728366 97.086325)))
+    (crossbar (pts (xy 125.731132 96.499911) (xy 178.731132 96.749911)))
+    (arrow1a (pts (xy 178.731132 96.749911) (xy 177.601875 97.331012)))
+    (arrow1b (pts (xy 178.731132 96.749911) (xy 177.607407 96.158183)))
+    (arrow2a (pts (xy 125.731132 96.499911) (xy 126.854857 97.091639)))
+    (arrow2b (pts (xy 125.731132 96.499911) (xy 126.860389 95.91881)))
+  )
+  (dimension 24.25 (width 0.15) (layer Dwgs.User)
+    (gr_text "0.9547 in" (at 185.3 80.625 270) (layer Dwgs.User)
+      (effects (font (size 1 1) (thickness 0.15)))
+    )
+    (feature1 (pts (xy 178.75 92.75) (xy 184.586421 92.75)))
+    (feature2 (pts (xy 178.75 68.5) (xy 184.586421 68.5)))
+    (crossbar (pts (xy 184 68.5) (xy 184 92.75)))
+    (arrow1a (pts (xy 184 92.75) (xy 183.413579 91.623496)))
+    (arrow1b (pts (xy 184 92.75) (xy 184.586421 91.623496)))
+    (arrow2a (pts (xy 184 68.5) (xy 183.413579 69.626504)))
+    (arrow2b (pts (xy 184 68.5) (xy 184.586421 69.626504)))
+  )
   (gr_text - (at 176 74.75) (layer F.SilkS)
     (effects (font (size 1 1) (thickness 0.15)))
@@
     (effects (font (size 1 1) (thickness 0.15)))
   )
-  (gr_line (start 125.75 68.25) (end 126.25 68.25) (layer Edge.Cuts) (width 0.05))
-  (gr_line (start 125.75 92.75) (end 125.75 68.25) (layer Edge.Cuts) (width 0.05))
-  (gr_line (start 134.75 92.75) (end 125.75 92.75) (layer Edge.Cuts) (width 0.05))
-  (gr_line (start 178.75 92.75) (end 134.75 92.75) (layer Edge.Cuts) (width 0.05))
-  (gr_line (start 178.75 68.5) (end 178.75 92.75) (layer Edge.Cuts) (width 0.05))
-  (gr_line (start 170.75 68.5) (end 178.75 68.5) (layer Edge.Cuts) (width 0.05))
-  (gr_line (start 170.75 73.75) (end 170.75 68.5) (layer Edge.Cuts) (width 0.05))
-  (gr_line (start 134.5 73.75) (end 170.75 73.75) (layer Edge.Cuts) (width 0.05))
-  (gr_line (start 134.5 68.25) (end 134.5 73.75) (layer Edge.Cuts) (width 0.05))
-  (gr_line (start 126.25 68.25) (end 134.5 68.25) (layer Edge.Cuts) (width 0.05))
+  (gr_line (start 125.75 68.25) (end 126.25 68.25) (layer Edge.Cuts) (width 0.4))
+  (gr_line (start 125.75 92.75) (end 125.75 68.25) (layer Edge.Cuts) (width 0.4))
+  (gr_line (start 134.75 92.75) (end 125.75 92.75) (layer Edge.Cuts) (width 0.4))
+  (gr_line (start 178.75 92.75) (end 134.75 92.75) (layer Edge.Cuts) (width 0.4))
+  (gr_line (start 178.75 68.5) (end 178.75 92.75) (layer Edge.Cuts) (width 0.4))
+  (gr_line (start 170.75 68.5) (end 178.75 68.5) (layer Edge.Cuts) (width 0.4))
+  (gr_line (start 170.75 73.75) (end 170.75 68.5) (layer Edge.Cuts) (width 0.4))
+  (gr_line (start 134.5 73.75) (end 170.75 73.75) (layer Edge.Cuts) (width 0.4))
+  (gr_line (start 134.5 68.25) (end 134.5 73.75) (layer Edge.Cuts) (width 0.4))
+  (gr_line (start 126.25 68.25) (end 134.5 68.25) (layer Edge.Cuts) (width 0.4))
   (dimension 42 (width 0.15) (layer Dwgs.User)
     (gr_text "42.000 mm" (at 152.75 66.95) (layer Dwgs.User)
@@
   (segment (start 137 89.55) (end 137.8 89.55) (width 1) (layer F.Cu) (net 6))
   (zone (net 2) (net_name GND) (layer B.Cu) (hatch edge 0.508)
-    (connect_pads (clearance 0.508))
+    (connect_pads (clearance 0.2))
     (min_thickness 0.254)
-    (fill yes (arc_segments 32) (thermal_gap 0.508) (thermal_bridge_width 1))
+    (fill yes (arc_segments 32) (thermal_gap 0.2) (thermal_bridge_width 0.75))
     (polygon
       (pts
@@
   )
   (zone (net 2) (net_name GND) (layer F.Cu) (hatch edge 0.508)
-    (connect_pads (clearance 0.508))
+    (connect_pads (clearance 0.2))
     (min_thickness 0.254)
-    (fill yes (arc_segments 32) (thermal_gap 0.508) (thermal_bridge_width 1))
+    (fill yes (arc_segments 32) (thermal_gap 0.2) (thermal_bridge_width 0.75))
     (polygon
       (pts
